File: Teste Rápido Fonte Chaveada.kicad_pcb (KiCad board)
At the start: 2 copper layers, 0 parts

Commit message: Atualização da placa v0.1 (@JefersonMarcante)
Parts:
- added CN1: W4505-20PDRDTXR, Library:W4505-20PDRDTXR, F.Cu at (120.5, 53.5)
- added D1: LED, Library:LED_1206_HandSolder, F.Cu at (108.7, 57.7)
- added D2: LED, Library:LED_1206_HandSolder, F.Cu at (108.7, 61.8)
- added D3: LED, Library:LED_1206_HandSolder, F.Cu at (108.7, 74.5)
- added D4: LED, Library:LED_1206_HandSolder, F.Cu at (108.7, 78.7)
- added D5: LED, Library:LED_1206_HandSolder, F.Cu at (108.7, 82.9)
- added D6: LED, Library:LED_1206_HandSolder, F.Cu at (108.7, 87.1)
- added D7: LED, Library:LED_1206_HandSolder, F.Cu at (108.7, 91.3)
- added R1: 100R, Library:RES_1206_HandSolder, F.Cu at (114.7, 57.7)
- added R2: 1k8R, Library:RES_1206_HandSolder, F.Cu at (114.7, 61.8)
- added R3: 470R, Library:RES_1206_HandSolder, F.Cu at (114.7, 74.5)
- added R4: 470R, Library:RES_1206_HandSolder, F.Cu at (114.7, 78.7)
- added R5: 470R, Library:RES_1206_HandSolder, F.Cu at (114.7, 82.9)
- added R6: 680R, Library:RES_1206_HandSolder, F.Cu at (114.7, 87.1)
- added R7: 1K8R, Library:RES_1206_HandSolder, F.Cu at (114.7, 91.3)
- added SW1: SW_DPST_x2, Library:SW_Push_1P1T_NO_6x6mm_H9.5mm, F.Cu at (111.7, 68.2)
Routing:
- net GND: track 0.00 -> 52.7 mm
- net /PS_ON: track 0.00 -> 20.1 mm
- net -5V: track 0.00 -> 11.5 mm
- net -12V: track 0.00 -> 11.5 mm
- net +P_G: track 0.00 -> 4.28 mm
- net +5V_SB: track 0.00 -> 4.28 mm
- net +5V: track 0.00 -> 4.28 mm
- net +3.3V: track 0.00 -> 4.28 mm
- net +12V: track 0.00 -> 4.28 mm
- net Net-(D7-A): track 0.00 -> 2.95 mm
- net Net-(D6-A): track 0.00 -> 2.95 mm
- net Net-(D5-A): track 0.00 -> 2.95 mm
- net Net-(D4-K): track 0.00 -> 2.95 mm
- net Net-(D3-A): track 0.00 -> 2.95 mm
- net Net-(D2-K): track 0.00 -> 2.95 mm
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Other:
- board outline added: 30 x 50 mm
- board text added: "+12V"
- board text added: "+3V3"
- board text added: "+5V"
- board text added: "+5VSB"
- board text added: "-12V"
- board text added: "-5V"
- board text added: "P.G."
- board text added: "PS_ON"
