File: Versão PTH/Teste Rápido Fonte Chaveada.kicad_sch (KiCad schematic)
At the start: 16 parts, among them CN1 W4505-20PDRDTXR, SW1 SW_DPST_x2

Commit message: Atualização da placa v1
Parts:
- D1: renamed from D5; footprint Library:LED_1206_HandSolder -> Library:LED_D3.0mm
- D2: renamed from D6; footprint Library:LED_1206_HandSolder -> Library:LED_D3.0mm
- D3: renamed from D7; footprint Library:LED_1206_HandSolder -> Library:LED_D3.0mm
- D4: renamed from D3; footprint Library:LED_1206_HandSolder -> Library:LED_D3.0mm
- D5: renamed from D1; footprint Library:LED_1206_HandSolder -> Library:LED_D3.0mm
- D6: renamed from D4; footprint Library:LED_1206_HandSolder -> Library:LED_D3.0mm
- D7: renamed from D2; footprint Library:LED_1206_HandSolder -> Library:LED_D3.0mm
- R1: renamed from R5; footprint Library:RES_1206_HandSolder -> Library:R_Axial_DIN0207_L6.3mm_D2.5mm_P10.16mm_Horizontal
- R2: renamed from R6; footprint Library:RES_1206_HandSolder -> Library:R_Axial_DIN0207_L6.3mm_D2.5mm_P10.16mm_Horizontal
- R3: renamed from R7; footprint Library:RES_1206_HandSolder -> Library:R_Axial_DIN0207_L6.3mm_D2.5mm_P10.16mm_Horizontal
- R4: renamed from R3; footprint Library:RES_1206_HandSolder -> Library:R_Axial_DIN0207_L6.3mm_D2.5mm_P10.16mm_Horizontal
- R5: renamed from R1; footprint Library:RES_1206_HandSolder -> Library:R_Axial_DIN0207_L6.3mm_D2.5mm_P10.16mm_Horizontal
- R6: renamed from R4; footprint Library:RES_1206_HandSolder -> Library:R_Axial_DIN0207_L6.3mm_D2.5mm_P10.16mm_Horizontal
- R7: renamed from R2; footprint Library:RES_1206_HandSolder -> Library:R_Axial_DIN0207_L6.3mm_D2.5mm_P10.16mm_Horizontal
- SW1: footprint Library:SW_Push_1P1T_NO_6x6mm_H9.5mm -> Library:SW_PUSH_6mm_H4.3mm
Changed lines of the file:
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@@
 		(dnp no)
 		(fields_autoplaced yes)
-		(property "Reference" "R5"
+		(property "Reference" "R1"
 			(at 158.75 105.4099 0)
 			(effects
@@
 			)
 		)
-		(property "Footprint" "Library:RES_1206_HandSolder"
+		(property "Footprint" "Library:R_Axial_DIN0207_L6.3mm_D2.5mm_P10.16mm_Horizontal"
 			(at 154.432 106.68 90)
 			(effects
@@
 			(project ""
 				(path "/05a0489b-6f48-4980-a6d7-922522b33b13"
-					(reference "R5")
+					(reference "R1")
 					(unit 1)
 				)
@@
 		(dnp no)
 		(fields_autoplaced yes)
-		(property "Reference" "R2"
+		(property "Reference" "R7"
 			(at 149.86 105.4099 0)
 			(effects
@@
 			)
 		)
-		(property "Footprint" "Library:RES_1206_HandSolder"
+		(property "Footprint" "Library:R_Axial_DIN0207_L6.3mm_D2.5mm_P10.16mm_Horizontal"
 			(at 145.542 106.68 90)
 			(effects
@@
 			(project "Teste Rápido Fonte Chaveada"
 				(path "/05a0489b-6f48-4980-a6d7-922522b33b13"
-					(reference "R2")
+					(reference "R7")
 					(unit 1)
 				)
@@
 		(dnp no)
 		(fields_autoplaced yes)
-		(property "Reference" "D7"
+		(property "Reference" "D3"
 			(at 132.08 115.8874 90)
 			(effects
@@
 			)
 		)
-		(property "Footprint" "Library:LED_1206_HandSolder"
+		(property "Footprint" "Library:LED_D3.0mm"
 			(at 128.27 115.57 0)
 			(effects
@@
 			(project "Teste Rápido Fonte Chaveada"
 				(path "/05a0489b-6f48-4980-a6d7-922522b33b13"
-					(reference "D7")
+					(reference "D3")
 					(unit 1)
 				)
@@
 		(dnp no)
 		(fields_autoplaced yes)
-		(property "Reference" "D2"
+		(property "Reference" "D7"
 			(at 150.1092 112.7124 90)
 			(effects
@@
 			)
 		)
-		(property "Footprint" "Library:LED_1206_HandSolder"
+		(property "Footprint" "Library:LED_D3.0mm"
 			(at 147.32 115.57 0)
 			(effects
@@
 			(project "Teste Rápido Fonte Chaveada"
 				(path "/05a0489b-6f48-4980-a6d7-922522b33b13"
-					(reference "D2")
+					(reference "D7")
 					(unit 1)
 				)
@@
 		(dnp no)
 		(fields_autoplaced yes)
-		(property "Reference" "R1"
+		(property "Reference" "R5"
 			(at 110.49 105.4099 0)
 			(effects
@@
 			)
 		)
-		(property "Footprint" "Library:RES_1206_HandSolder"
+		(property "Footprint" "Library:R_Axial_DIN0207_L6.3mm_D2.5mm_P10.16mm_Horizontal"
 			(at 106.172 106.68 90)
 			(effects
@@
 			(project "Teste Rápido Fonte Chaveada"
 				(path "/05a0489b-6f48-4980-a6d7-922522b33b13"
-					(reference "R1")
+					(reference "R5")
 					(unit 1)
 				)
@@
 		(dnp no)
 		(fields_autoplaced yes)
-		(property "Reference" "R6"
+		(property "Reference" "R2"
 			(at 100.33 105.4099 0)
 			(effects
@@
 			)
 		)
-		(property "Footprint" "Library:RES_1206_HandSolder"
+		(property "Footprint" "Library:R_Axial_DIN0207_L6.3mm_D2.5mm_P10.16mm_Horizontal"
 			(at 96.012 106.68 90)
 			(effects
@@
 			(project "Teste Rápido Fonte Chaveada"
 				(path "/05a0489b-6f48-4980-a6d7-922522b33b13"
-					(reference "R6")
+					(reference "R2")
 					(unit 1)
 				)
@@
 		(dnp no)
 		(fields_autoplaced yes)
-		(property "Reference" "D5"
+		(property "Reference" "D1"
 			(at 160.02 115.8874 90)
 			(effects
@@
 			)
 		)
-		(property "Footprint" "Library:LED_1206_HandSolder"
+		(property "Footprint" "Library:LED_D3.0mm"
 			(at 156.21 115.57 0)
 			(effects
@@
 			(project "Teste Rápido Fonte Chaveada"
 				(path "/05a0489b-6f48-4980-a6d7-922522b33b13"
-					(reference "D5")
+					(reference "D1")
 					(unit 1)
 				)
@@
 		(dnp no)
 		(fields_autoplaced yes)
-		(property "Reference" "D4"
+		(property "Reference" "D6"
 			(at 140.97 112.7124 90)
 			(effects
@@
 			)
 		)
-		(property "Footprint" "Library:LED_1206_HandSolder"
+		(property "Footprint" "Library:LED_D3.0mm"
 			(at 138.43 115.57 0)
 			(effects
@@
 			(project "Teste Rápido Fonte Chaveada"
 				(path "/05a0489b-6f48-4980-a6d7-922522b33b13"
-					(reference "D4")
+					(reference "D6")
 					(unit 1)
 				)
@@
 		(dnp no)
 		(fields_autoplaced yes)
-		(property "Reference" "D1"
+		(property "Reference" "D5"
 			(at 111.76 115.8874 90)
 			(effects
@@
 			)
 		)
-		(property "Footprint" "Library:LED_1206_HandSolder"
+		(property "Footprint" "Library:LED_D3.0mm"
 			(at 107.95 115.57 0)
 			(effects
@@
 			(project "Teste Rápido Fonte Chaveada"
 				(path "/05a0489b-6f48-4980-a6d7-922522b33b13"
-					(reference "D1")
+					(reference "D5")
 					(unit 1)
 				)
@@
 		(dnp no)
 		(fields_autoplaced yes)
-		(property "Reference" "R4"
+		(property "Reference" "R6"
 			(at 140.97 105.4099 0)
 			(effects
@@
 			)
 		)
-		(property "Footprint" "Library:RES_1206_HandSolder"
+		(property "Footprint" "Library:R_Axial_DIN0207_L6.3mm_D2.5mm_P10.16mm_Horizontal"
 			(at 136.652 106.68 90)
 			(effects
@@
 			(project "Teste Rápido Fonte Chaveada"
 				(path "/05a0489b-6f48-4980-a6d7-922522b33b13"
-					(reference "R4")
+					(reference "R6")
 					(unit 1)
 				)
@@
 			)
 		)
-		(property "Footprint" "Library:SW_Push_1P1T_NO_6x6mm_H9.5mm"
+		(property "Footprint" "Library:SW_PUSH_6mm_H4.3mm"
 			(at 88.9 105.41 0)
 			(effects
@@
 		(dnp no)
 		(fields_autoplaced yes)
-		(property "Reference" "D3"
+		(property "Reference" "D4"
 			(at 121.92 115.8874 90)
 			(effects
@@
 			)
 		)
-		(property "Footprint" "Library:LED_1206_HandSolder"
+		(property "Footprint" "Library:LED_D3.0mm"
 			(at 118.11 115.57 0)
 			(effects
@@
 			(project "Teste Rápido Fonte Chaveada"
 				(path "/05a0489b-6f48-4980-a6d7-922522b33b13"
-					(reference "D3")
+					(reference "D4")
 					(unit 1)
 				)
@@
 		(dnp no)
 		(fields_autoplaced yes)
-		(property "Reference" "R7"
+		(property "Reference" "R3"
 			(at 130.81 105.4099 0)
 			(effects
@@
 			)
 		)
-		(property "Footprint" "Library:RES_1206_HandSolder"
+		(property "Footprint" "Library:R_Axial_DIN0207_L6.3mm_D2.5mm_P10.16mm_Horizontal"
 			(at 126.492 106.68 90)
 			(effects
@@
 			(project "Teste Rápido Fonte Chaveada"
 				(path "/05a0489b-6f48-4980-a6d7-922522b33b13"
-					(reference "R7")
+					(reference "R3")
 					(unit 1)
 				)
@@
 		(dnp no)
 		(fields_autoplaced yes)
-		(property "Reference" "R3"
+		(property "Reference" "R4"
 			(at 120.65 105.4099 0)
 			(effects
@@
 			)
 		)
-		(property "Footprint" "Library:RES_1206_HandSolder"
+		(property "Footprint" "Library:R_Axial_DIN0207_L6.3mm_D2.5mm_P10.16mm_Horizontal"
 			(at 116.332 106.68 90)
 			(effects
@@
 			(project "Teste Rápido Fonte Chaveada"
 				(path "/05a0489b-6f48-4980-a6d7-922522b33b13"
-					(reference "R3")
+					(reference "R4")
 					(unit 1)
 				)
@@
 		(dnp no)
 		(fields_autoplaced yes)
-		(property "Reference" "D6"
+		(property "Reference" "D2"
 			(at 101.6 115.8874 90)
 			(effects
@@
 			)
 		)
-		(property "Footprint" "Library:LED_1206_HandSolder"
+		(property "Footprint" "Library:LED_D3.0mm"
 			(at 97.79 115.57 0)
 			(effects
@@
 			(project ""
 				(path "/05a0489b-6f48-4980-a6d7-922522b33b13"
-					(reference "D6")
-					(unit 1)
-				)
+					(reference "D2")
+					(unit 1)
+				)
